Commit message: feat: Remap IMU and LiDAR topics and frames to the `livox` namespace and disable default state estimation nodes.

File: champ/champ_description/urdf/accessories.urdf.xacro (robot description, xacro)
@@ -19,5 +19,5 @@
             <origin xyz="${base_length / 2} 0.0 -${base_height / 2 + 0.01}" rpy="0 0 0"/>
         </xacro:asus_camera>
-        <link name="imu_link">
+        <link name="livox_frame">
             <inertial>
                 <mass value="0.001"/>
@@ -28,7 +28,7 @@
         <joint name="imu_joint" type="fixed">
             <parent link="${base_name}" />
-            <child link="imu_link" />
+            <child link="livox_frame" />
         </joint>
-        <gazebo reference="imu_link">
+        <gazebo reference="livox_frame">
                 <sensor name="imu_controller" type="imu">
                     <always_on>true</always_on>
@@ -36,10 +36,10 @@
                     <plugin name="gazebo_ros_imu_sensor" filename="libgazebo_ros_imu_sensor.so">
                         <ros>
-                            <namespace>/imu</namespace>
-                            <argument>~/out:=data</argument>
+                            <namespace>livox</namespace>
+                            <argument>~/out:=imu</argument>
                         </ros>
                         <!-- <updateRate>50.0</updateRate>
                         <bodyName>imu_link</bodyName>
-                        <topicName>imu/data</topicName>
+                        <topicName>livox/imu</topicName>
                         <accelDrift>0.005 0.005 0.005</accelDrift>
                         <accelGaussianNoise>0.005 0.005 0.005</accelGaussianNoise>

File: robots/descriptions/go2_description/xacro/gazebo.xacro (robot description, xacro)
@@ -19,5 +19,5 @@
       </plugin>
     </gazebo>
-    <gazebo reference="imu_link">
+    <gazebo reference="livox_frame">
         <sensor name="imu_sensor" type="imu">
             <always_on>true</always_on>
@@ -67,6 +67,6 @@
             <plugin name="imu_plugin" filename="libgazebo_ros_imu_sensor.so">
                 <ros>
-                    <namespace>imu</namespace>
-                    <remapping>~/out:=data</remapping>
+                    <namespace>livox</namespace>
+                    <remapping>~/out:=imu</remapping>
                 </ros>
                 <initial_orientation_as_reference>false</initial_orientation_as_reference>

File: robots/descriptions/go2_description/xacro/robot_VLP.xacro (robot description, xacro)
@@ -58,8 +58,8 @@
     <joint name="imu_joint" type="fixed">
         <parent link="trunk"/>
-        <child link="imu_link"/>
+        <child link="livox_frame"/>
         <origin rpy="0 0 0" xyz="0 0 0"/>
     </joint>
-    <link name="imu_link">
+    <link name="livox_frame">
         <inertial>
             <mass value="0.001"/>

File: robots/descriptions/go2_description/xacro/velodyne.xacro (robot description, xacro)
@@ -82,7 +82,7 @@
             <ros>
               <namespace>/</namespace>
-              <remapping>~/out:=velodyne_points</remapping>
+              <remapping>~/out:=livox/lidar</remapping>
             </ros>
-            <frame_name>velodyne</frame_name>
+            <frame_name>livox_frame</frame_name>
             <organize_cloud>false</organize_cloud>
             <min_range>0.9</min_range>
